File: PCBs/early_energy_test_PCB/energy_test_PCB/energy_test_PCB.kicad_sch (KiCad schematic)
At the start: 31 parts, among them J1 B2B-PH-K-S_LF__SN_, J2 B2B-PH-K-S_LF__SN_, J3 B2B-PH-K-S_LF__SN_, U1 IRLML6244TRPBF, U3 LTC4071EMS8E_PBF

Commit message: Add receiver PCB files and update energy test PCB (V0)
Added new receiver PCB design files, including footprints, symbols, 3D models, and project backups. Updated early energy test PCB files with detailed board layout and schematic content.
Parts:
- C1, C10, C11, C12, C2, C3, C4, C5, C6, C7, C8, C9, R1, R2, R3, R4, R5, R6, R7, R8, TH1: footprint (none) -> Resistor_THT:R_Axial_DIN0207_L6.3mm_D2.5mm_P7.62mm_Horizontal
- D1, D2: footprint SMD-DIODE-SCHOTTKY-40V-1A_DO-214AC_:DO-214AC -> Resistor_THT:R_Axial_DIN0207_L6.3mm_D2.5mm_P7.62mm_Horizontal
- J1, J2, J3: footprint B2B-PH-K-S_LF__SN_:JST_B2B-PH-K-S_LF__SN_ -> PCB_footprints:JST_B2B-PH-K-S_LF__SN_
- L1, L2: footprint (none) -> Inductor_THT:L_Radial_D12.0mm_P10.00mm_Neosid_SD12_style1
- U1: footprint IRLML6244TRPBF:SOT95P237X112-3N -> PCB_footprints:SOT95P237X112-3N
- U3: footprint LTC4071EMS8E_PBF:MSOP-8_MS -> PCB_footprints:MSOP-8_MS
- VR1: footprint MCP1700T-3302E_TT:SOT95P237X112-3N -> PCB_footprints:SOT95P237X112-3N
Changed lines of the file:
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@@
 	)
 	(junction
-		(at 29.21 58.42)
+		(at 40.64 68.58)
 		(diameter 0)
 		(color 0 0 0 0)
 	)
 	(junction
-		(at 40.64 68.58)
+		(at 184.15 30.48)
 		(diameter 0)
 		(color 0 0 0 0)
 	)
 	(junction
-		(at 184.15 30.48)
+		(at 29.21 66.04)
 		(diameter 0)
 		(color 0 0 0 0)
@@
 	)
 	(junction
-		(at 29.21 66.04)
-		(diameter 0)
-		(color 0 0 0 0)
-	)
-	(junction
 		(at 137.16 38.1)
 		(diameter 0)
@@
 	)
 	(junction
+		(at 29.21 58.42)
+		(diameter 0)
+		(color 0 0 0 0)
+	)
+	(junction
 		(at 184.15 38.1)
 		(diameter 0)
@@
 	(wire
 		(pts
+			(xy 29.21 66.04) (xy 31.75 66.04)
+		)
+		(stroke
+			(width 0)
+			(type default)
+		)
+	)
+	(wire
+		(pts
 			(xy 124.46 30.48) (xy 124.46 49.53)
 		)
@@
 	(wire
 		(pts
-			(xy 29.21 58.42) (xy 41.91 58.42)
-		)
-		(stroke
-			(width 0)
-			(type default)
-		)
-	)
-	(wire
-		(pts
 			(xy 54.61 33.02) (xy 54.61 35.56)
 		)
@@
 	(wire
 		(pts
-			(xy 184.15 38.1) (xy 190.5 38.1)
+			(xy 29.21 58.42) (xy 41.91 58.42)
 		)
 		(stroke
@@
 	(wire
 		(pts
-			(xy 173.99 43.18) (xy 176.53 43.18)
+			(xy 184.15 38.1) (xy 190.5 38.1)
 		)
 		(stroke
@@
 	(wire
 		(pts
-			(xy 120.65 38.1) (xy 120.65 39.37)
+			(xy 173.99 43.18) (xy 176.53 43.18)
 		)
 		(stroke
@@
 	(wire
 		(pts
-			(xy 29.21 66.04) (xy 31.75 66.04)
+			(xy 120.65 38.1) (xy 120.65 39.37)
 		)
 		(stroke
@@
 			)
 		)
-		(property "Footprint" "LTC4071EMS8E_PBF:MSOP-8_MS"
+		(property "Footprint" "PCB_footprints:MSOP-8_MS"
 			(at 41.91 58.42 0)
 			(effects
@@
 			)
 		)
-		(property "Footprint" ""
+		(property "Footprint" "Resistor_THT:R_Axial_DIN0207_L6.3mm_D2.5mm_P7.62mm_Horizontal"
 			(at 138.1252 38.1 0)
 			(effects
@@
 			)
 		)
-		(property "Footprint" ""
+		(property "Footprint" "Resistor_THT:R_Axial_DIN0207_L6.3mm_D2.5mm_P7.62mm_Horizontal"
 			(at 39.6748 68.58 0)
 			(effects
@@
 			)
 		)
-		(property "Footprint" ""
+		(property "Footprint" "Resistor_THT:R_Axial_DIN0207_L6.3mm_D2.5mm_P7.62mm_Horizontal"
 			(at 121.6152 38.1 0)
 			(effects
@@
 		(on_board yes)
 		(dnp no)
-		(fields_autoplaced yes)
 		(property "Reference" "J3"
-			(at 212.09 38.0999 0)
+			(at 200.914 45.466 0)
 			(effects
 				(font
@@
 		)
 		(property "Value" "B2B-PH-K-S_LF__SN_"
-			(at 212.09 40.6399 0)
+			(at 200.914 48.006 0)
 			(effects
 				(font
@@
 			)
 		)
-		(property "Footprint" "B2B-PH-K-S_LF__SN_:JST_B2B-PH-K-S_LF__SN_"
+		(property "Footprint" "PCB_footprints:JST_B2B-PH-K-S_LF__SN_"
 			(at 204.47 40.64 0)
 			(effects
@@
 		)
 		(property "Value" "SMD-DIODE-SCHOTTKY-40V-1A_DO-214AC_"
-			(at 139.192 42.164 0)
+			(at 132.842 40.64 0)
 			(effects
 				(font
@@
 			)
 		)
-		(property "Footprint" "SMD-DIODE-SCHOTTKY-40V-1A_DO-214AC_:DO-214AC"
+		(property "Footprint" "Resistor_THT:R_Axial_DIN0207_L6.3mm_D2.5mm_P7.62mm_Horizontal"
 			(at 132.08 38.1 0)
 			(effects
@@
 			)
 		)
-		(property "Footprint" ""
+		(property "Footprint" "Resistor_THT:R_Axial_DIN0207_L6.3mm_D2.5mm_P7.62mm_Horizontal"
 			(at 47.9552 35.56 0)
 			(effects
@@
 			)
 		)
-		(property "Footprint" ""
+		(property "Footprint" "Resistor_THT:R_Axial_DIN0207_L6.3mm_D2.5mm_P7.62mm_Horizontal"
 			(at 22.86 60.198 90)
 			(effects
@@
 			)
 		)
-		(property "Footprint" ""
+		(property "Footprint" "Resistor_THT:R_Axial_DIN0207_L6.3mm_D2.5mm_P7.62mm_Horizontal"
 			(at 19.558 62.23 90)
 			(effects
@@
 			)
 		)
-		(property "Footprint" ""
+		(property "Footprint" "Resistor_THT:R_Axial_DIN0207_L6.3mm_D2.5mm_P7.62mm_Horizontal"
 			(at 177.4952 50.8 0)
 			(effects
@@
 			)
 		)
-		(property "Footprint" ""
+		(property "Footprint" "Inductor_THT:L_Radial_D12.0mm_P10.00mm_Neosid_SD12_style1"
 			(at 111.76 30.48 0)
 			(effects
@@
 			)
 		)
-		(property "Footprint" "B2B-PH-K-S_LF__SN_:JST_B2B-PH-K-S_LF__SN_"
+		(property "Footprint" "PCB_footprints:JST_B2B-PH-K-S_LF__SN_"
 			(at 128.27 20.32 0)
 			(effects
@@
 			)
 		)
-		(property "Footprint" ""
+		(property "Footprint" "Resistor_THT:R_Axial_DIN0207_L6.3mm_D2.5mm_P7.62mm_Horizontal"
 			(at 140.208 73.66 90)
 			(effects
@@
 			)
 		)
-		(property "Footprint" "SMD-DIODE-SCHOTTKY-40V-1A_DO-214AC_:DO-214AC"
+		(property "Footprint" "Resistor_THT:R_Axial_DIN0207_L6.3mm_D2.5mm_P7.62mm_Horizontal"
 			(at 58.42 38.1 0)
 			(effects
@@
 			)
 		)
-		(property "Footprint" ""
+		(property "Footprint" "Inductor_THT:L_Radial_D12.0mm_P10.00mm_Neosid_SD12_style1"
 			(at 58.42 33.02 0)
 			(effects
@@
 			)
 		)
-		(property "Footprint" ""
+		(property "Footprint" "Resistor_THT:R_Axial_DIN0207_L6.3mm_D2.5mm_P7.62mm_Horizontal"
 			(at 40.3352 35.56 0)
 			(effects
@@
 			)
 		)
-		(property "Footprint" ""
+		(property "Footprint" "Resistor_THT:R_Axial_DIN0207_L6.3mm_D2.5mm_P7.62mm_Horizontal"
 			(at 178.7652 38.1 0)
 			(effects
@@
 		(dnp no)
 		(property "Reference" "C10"
-			(at 43.18 60.9599 0)
+			(at 32.258 61.214 0)
 			(effects
 				(font
@@
 		)
 		(property "Value" "C"
-			(at 33.02 63.4999 0)
+			(at 27.178 64.008 0)
 			(effects
 				(font
@@
 			)
 		)
-		(property "Footprint" ""
+		(property "Footprint" "Resistor_THT:R_Axial_DIN0207_L6.3mm_D2.5mm_P7.62mm_Horizontal"
 			(at 28.2448 58.42 0)
 			(effects
@@
 			)
 		)
-		(property "Footprint" "IRLML6244TRPBF:SOT95P237X112-3N"
+		(property "Footprint" "PCB_footprints:SOT95P237X112-3N"
 			(at 86.36 35.56 0)
 			(effects
@@
 		(dnp no)
 		(property "Reference" "C12"
-			(at 134.62 60.9599 0)
+			(at 122.174 59.944 0)
 			(effects
 				(font
@@
 			)
 		)
-		(property "Footprint" ""
+		(property "Footprint" "Resistor_THT:R_Axial_DIN0207_L6.3mm_D2.5mm_P7.62mm_Horizontal"
 			(at 119.6848 58.42 0)
 			(effects
@@
 		(on_board yes)
 		(dnp no)
-		(fields_autoplaced yes)
 		(property "Reference" "R6"
-			(at 127 59.69 90)
+			(at 128.524 64.262 90)
 			(effects
 				(font
@@
 			)
 		)
-		(property "Footprint" ""
+		(property "Footprint" "Resistor_THT:R_Axial_DIN0207_L6.3mm_D2.5mm_P7.62mm_Horizontal"
 			(at 127 67.818 90)
 			(effects
@@
 			)
 		)
-		(property "Footprint" "MCP1700T-3302E_TT:SOT95P237X112-3N"
+		(property "Footprint" "PCB_footprints:SOT95P237X112-3N"
 			(at 156.21 40.64 0)
 			(effects
@@
 			)
 		)
-		(property "Footprint" ""
+		(property "Footprint" "Resistor_THT:R_Axial_DIN0207_L6.3mm_D2.5mm_P7.62mm_Horizontal"
 			(at 185.1152 38.1 0)
 			(effects
@@
 		(on_board yes)
 		(dnp no)
-		(fields_autoplaced yes)
 		(property "Reference" "#PWR04"
 			(at 120.65 45.72 0)
@@
 		)
 		(property "Value" "GND"
-			(at 120.65 44.45 0)
+			(at 121.666 41.91 0)
 			(effects
 				(font
@@
 			)
 		)
-		(property "Footprint" ""
+		(property "Footprint" "Resistor_THT:R_Axial_DIN0207_L6.3mm_D2.5mm_P7.62mm_Horizontal"
 			(at 115.062 45.72 90)
 			(effects
@@
 			)
 		)
-		(property "Footprint" ""
+		(property "Footprint" "Resistor_THT:R_Axial_DIN0207_L6.3mm_D2.5mm_P7.62mm_Horizontal"
 			(at 140.208 62.23 90)
 			(effects
@@
 		(on_board yes)
 		(dnp no)
-		(fields_autoplaced yes)
 		(property "Reference" "R5"
-			(at 31.75 62.23 90)
+			(at 32.258 71.12 90)
 			(effects
 				(font
@@
 		)
 		(property "Value" "R"
-			(at 31.75 64.77 90)
+			(at 30.734 68.58 90)
 			(effects
 				(font
@@
 			)
 		)
-		(property "Footprint" ""
+		(property "Footprint" "Resistor_THT:R_Axial_DIN0207_L6.3mm_D2.5mm_P7.62mm_Horizontal"
 			(at 31.75 66.802 90)
 			(effects
@@
 			)
 		)
-		(property "Footprint" ""
+		(property "Footprint" "Resistor_THT:R_Axial_DIN0207_L6.3mm_D2.5mm_P7.62mm_Horizontal"
 			(at 144.78 68.58 0)
 			(effects
@@
 			)
 		)
-		(property "Footprint" ""
+		(property "Footprint" "Resistor_THT:R_Axial_DIN0207_L6.3mm_D2.5mm_P7.62mm_Horizontal"
 			(at 38.608 72.39 90)
 			(effects
@@
 			)
 		)
-		(property "Footprint" ""
+		(property "Footprint" "Resistor_THT:R_Axial_DIN0207_L6.3mm_D2.5mm_P7.62mm_Horizontal"
 			(at 191.4652 38.1 0)
 			(effects
@@
 			)
 		)
-		(property "Footprint" "B2B-PH-K-S_LF__SN_:JST_B2B-PH-K-S_LF__SN_"
+		(property "Footprint" "PCB_footprints:JST_B2B-PH-K-S_LF__SN_"
 			(at 24.13 35.56 0)
 			(effects
@@
 		(on_board yes)
 		(dnp no)
-		(fields_autoplaced yes)
 		(property "Reference" "C9"
-			(at 77.47 41.91 90)
+			(at 81.534 52.324 90)
 			(effects
 				(font
@@
 			)
 		)
-		(property "Footprint" ""
+		(property "Footprint" "Resistor_THT:R_Axial_DIN0207_L6.3mm_D2.5mm_P7.62mm_Horizontal"
 			(at 81.28 48.5648 0)
 			(effects
