File: PCBs/receiver_PCB/receiver/receiver.kicad_sch (KiCad schematic)
At the start: 12 parts, among them U1 NRF54L15-CAAA-R

Commit message: Add soft_nRF_R project and update receiver PCB
Added new soft_nRF_R firmware project with initial source files. Updated receiver PCB design to use Wurth Elektronik connectors, revised net assignments, and replaced legacy footprints. Adjusted .gitignore for new build directory. Minor updates to other PCB and source files for consistency.
Parts:
- removed U1: NRF54L15-CAAA-R, PCB_footprints:BGA47N30P7X7_245X224X46N, symbol NRF54L15-CAAA-R:NRF54L15-CAAA-R
- added J1, J2, J3, J4, J5: 6570XX140201_657002140201, PCB_footprints_connector:657002140201, symbol 6570XX140201_657002140201:6570XX140201_657002140201
Connections:
- net GND: now also J1.1, J1.2
- net at C1.2, C2.1, D1.A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: now also J2.1, J2.2
- net at LS1.N: now also J5.1, J5.2
- net at R2.1: now also J3.1, J3.2
- net at R1.1: now also J4.1, J4.2
